Commit message: Adicion de avance

File: catkin_ws/src/mechdog_description/urdf/mechdog.urdf.xacro (robot description, xacro)
@@ -193,11 +193,10 @@
   </xacro:unless>
   <xacro:if eval="$(arg simulation)">
-    <gazebo>
-      <!-- Ground plane -->
-      <static>true</static>
-    </gazebo>
     <!-- LIDAR Sensor Plugin -->
     <gazebo reference="lidar_link">
+      <material>Gazebo/Black</material>
       <sensor type="ray" name="lidar_sensor">
+        <pose>0 0 0 0 0 0</pose>
+        <visualize>true</visualize>
         <update_rate>20</update_rate>
         <ray>
@@ -211,15 +210,17 @@
           </scan>
           <range>
-            <min>0.1</min>
+            <min>0.10</min>
             <max>10.0</max>
             <resolution>0.01</resolution>
           </range>
+          <noise>
+            <type>gaussian</type>
+            <mean>0.0</mean>
+            <stddev>0.001</stddev>
+          </noise>
         </ray>
-        <plugin name="gazebo_ros_base_sensor" filename="libgazebo_ros_base_sensor.so">
-          <ros>
-            <namespace>/mechdog</namespace>
-            <remapping>~/out:=scan</remapping>
-          </ros>
-          <outputType>sensor_msgs/LaserScan</outputType>
+        <plugin name="gazebo_ros_laser_controller" filename="libgazebo_ros_laser.so">
+          <topicName>/gazebo/lidar_clean</topicName>
+          <frameName>lidar_link</frameName>
         </plugin>
       </sensor>
@@ -227,3 +228,2 @@
   </xacro:if>
 </robot>
-EOF

Commit message: no se jefe estoy cansado

File: catkin_ws/src/mechdog_description/urdf/mechdog.urdf.xacro (robot description, xacro)
@@ -1,4 +1,5 @@
 <?xml version="1.0"?>
 <robot name="mechdog" xmlns:xacro="http://www.ros.org/wiki/xacro">
+  <xacro:arg name="simulation" default="false"/>
   <!-- Robot Properties -->
   <xacro:property name="robot_length" value="0.5"/>
@@ -6,6 +7,7 @@
   <xacro:property name="robot_height" value="0.2"/>
   <xacro:property name="robot_mass" value="15.0"/>
-  <!-- Sensor Offsets -->
-  <xacro:property name="lidar_offset_x" value="0.2"/>
+  <!-- Sensor Offsets — LIDAR placed just past the front legs (robot_length/2 = 0.25 m)
+       so that forward-facing rays do not hit the robot's own legs. -->
+  <xacro:property name="lidar_offset_x" value="0.28"/>
   <xacro:property name="lidar_offset_z" value="0.15"/>
   <!-- Velocity Limits -->
@@ -189,8 +191,22 @@
   </joint>
   <!-- Gazebo Plugins (conditioned on simulation) -->
-  <xacro:unless eval="$(arg simulation)">
+  <xacro:unless value="$(arg simulation)">
     <!-- Empty tag when not in simulation -->
   </xacro:unless>
-  <xacro:if eval="$(arg simulation)">
+  <xacro:if value="$(arg simulation)">
+    <!-- Ground-truth Odometry Plugin (P3D)
+         Publishes the robot's pose from Gazebo directly to /gazebo/odom_clean.
+         This is the source of truth consumed by noise_injector → /mechdog/odom. -->
+    <gazebo>
+      <plugin name="gazebo_ros_ground_truth_odom" filename="libgazebo_ros_p3d.so">
+        <bodyName>base_link</bodyName>
+        <topicName>/gazebo/odom_clean</topicName>
+        <frameName>world</frameName>
+        <xyzOffsets>0 0 0</xyzOffsets>
+        <rpyOffsets>0 0 0</rpyOffsets>
+        <updateRate>50.0</updateRate>
+        <gaussianNoise>0.0</gaussianNoise>
+      </plugin>
+    </gazebo>
     <!-- LIDAR Sensor Plugin -->
     <gazebo reference="lidar_link">

Commit message: abstraccion de sensor I2C no lidar como esta planteado

File: catkin_ws/src/mechdog_description/urdf/mechdog.urdf.xacro (robot description, xacro)
@@ -7,8 +7,10 @@
   <xacro:property name="robot_height" value="0.2"/>
   <xacro:property name="robot_mass" value="15.0"/>
-  <!-- Sensor Offsets — LIDAR placed just past the front legs (robot_length/2 = 0.25 m)
-       so that forward-facing rays do not hit the robot's own legs. -->
-  <xacro:property name="lidar_offset_x" value="0.28"/>
-  <xacro:property name="lidar_offset_z" value="0.15"/>
+  <!-- Sensor Offsets — Ultrasonic at front-center, past the legs -->
+  <xacro:property name="ultrasonic_offset_x" value="0.28"/>
+  <xacro:property name="ultrasonic_offset_z" value="0.15"/>
+  <xacro:property name="ultrasonic_fov" value="0.26"/>
+  <xacro:property name="ultrasonic_min_range" value="0.02"/>
+  <xacro:property name="ultrasonic_max_range" value="3.0"/>
   <!-- Velocity Limits -->
   <xacro:property name="max_velocity" value="1.0"/>
@@ -58,9 +60,9 @@
     <child link="base_link"/>
   </joint>
-  <!-- LIDAR Sensor -->
-  <link name="lidar_link">
-    <visual>
-      <geometry>
-        <cylinder length="0.1" radius="0.05"/>
+  <!-- Ultrasonic Sensor (HC-SR04 equivalent) -->
+  <link name="ultrasonic_link">
+    <visual>
+      <geometry>
+        <box size="0.02 0.02 0.01"/>
       </geometry>
       <material name="black"/>
@@ -68,19 +70,19 @@
     <collision>
       <geometry>
-        <cylinder length="0.1" radius="0.05"/>
-      </geometry>
-    </collision>
-    <inertial>
-      <mass value="0.1"/>
+        <box size="0.02 0.02 0.01"/>
+      </geometry>
+    </collision>
+    <inertial>
+      <mass value="0.01"/>
       <origin xyz="0 0 0" />
-      <inertia  ixx="0.0001" ixy="0.0" ixz="0.0"
-                iyy="0.0001" iyz="0.0" izz="0.0001"/>
-    </inertial>
-  </link>
-  <!-- Static transform from base_link to lidar_link -->
-  <joint name="base_link_lidar_link" type="fixed">
-    <origin xyz="${lidar_offset_x} 0 ${lidar_offset_z}" rpy="0 0 0"/>
-    <parent link="base_link"/>
-    <child link="lidar_link"/>
+      <inertia  ixx="0.00001" ixy="0.0" ixz="0.0"
+                iyy="0.00001" iyz="0.0" izz="0.00001"/>
+    </inertial>
+  </link>
+  <!-- Static transform from base_link to ultrasonic_link -->
+  <joint name="base_link_ultrasonic_link" type="fixed">
+    <origin xyz="${ultrasonic_offset_x} 0 ${ultrasonic_offset_z}" rpy="0 0 0"/>
+    <parent link="base_link"/>
+    <child link="ultrasonic_link"/>
   </joint>
   <!-- Simplified Leg Links (for visualization) -->
@@ -190,12 +192,7 @@
     <child link="leg_rear_right"/>
   </joint>
-  <!-- Gazebo Plugins (conditioned on simulation) -->
-  <xacro:unless value="$(arg simulation)">
-    <!-- Empty tag when not in simulation -->
-  </xacro:unless>
+  <!-- Simulation-only plugins (Gazebo) -->
   <xacro:if value="$(arg simulation)">
-    <!-- Ground-truth Odometry Plugin (P3D)
-         Publishes the robot's pose from Gazebo directly to /gazebo/odom_clean.
-         This is the source of truth consumed by noise_injector → /mechdog/odom. -->
+    <!-- Ground-truth Odometry Plugin (P3D) -->
     <gazebo>
       <plugin name="gazebo_ros_ground_truth_odom" filename="libgazebo_ros_p3d.so">
@@ -209,8 +206,9 @@
       </plugin>
     </gazebo>
-    <!-- LIDAR Sensor Plugin -->
-    <gazebo reference="lidar_link">
-      <material>Gazebo/Black</material>
-      <sensor type="ray" name="lidar_sensor">
+    <!-- Ultrasonic Range Sensor (HC-SR04 emulation)
+         Topic: /gazebo/ultrasonic_clean  (sensor_msgs/Range)
+         Max range: 3.0 m, FOV: 0.26 rad (15°), Rate: 20 Hz -->
+    <gazebo reference="ultrasonic_link">
+      <sensor type="ray" name="ultrasonic_sensor">
         <pose>0 0 0 0 0 0</pose>
         <visualize>true</visualize>
@@ -219,13 +217,13 @@
           <scan>
             <horizontal>
-              <samples>360</samples>
+              <samples>1</samples>
               <resolution>1</resolution>
-              <min_angle>-3.14159</min_angle>
-              <max_angle>3.14159</max_angle>
+              <min_angle>-0.13</min_angle>
+              <max_angle>0.13</max_angle>
             </horizontal>
           </scan>
           <range>
-            <min>0.10</min>
-            <max>10.0</max>
+            <min>0.02</min>
+            <max>3.0</max>
             <resolution>0.01</resolution>
           </range>
@@ -233,10 +231,16 @@
             <type>gaussian</type>
             <mean>0.0</mean>
-            <stddev>0.001</stddev>
+            <stddev>0.005</stddev>
           </noise>
         </ray>
-        <plugin name="gazebo_ros_laser_controller" filename="libgazebo_ros_laser.so">
-          <topicName>/gazebo/lidar_clean</topicName>
-          <frameName>lidar_link</frameName>
+        <plugin name="ultrasonic_range_controller" filename="libgazebo_ros_range.so">
+          <topicName>/gazebo/ultrasonic_clean</topicName>
+          <frameName>ultrasonic_link</frameName>
+          <radiationType>ultrasonic</radiationType>
+          <fov>0.26</fov>
+          <minDistance>0.02</minDistance>
+          <maxDistance>3.0</maxDistance>
+          <gaussianNoise>0.005</gaussianNoise>
+          <updateRate>20</updateRate>
         </plugin>
       </sensor>

File: catkin_ws/src/mechdog_description/urdf/mechdog_gazebo.xacro (robot description, xacro)
@@ -1,4 +1,7 @@
 <?xml version="1.0"?>
-<!-- Macro-only xacro: do not wrap in <robot> (included inside mechdog.urdf.xacro). -->
+<!-- mechdog_gazebo.xacro – Included by mechdog.urdf.xacro when simulation:=true
+     Usage in main URDF:
+       <xacro:include filename="$(find mechdog_description)/urdf/mechdog_gazebo.xacro"/>
+       <xacro:mechdog_gazebo_extensions prefix="" simulation="$(arg simulation)"/> -->
 <xacro:macro xmlns:xacro="http://www.ros.org/wiki/xacro" name="mechdog_gazebo_extensions" params="prefix simulation:=false">
   <xacro:if value="${simulation}">
@@ -8,6 +11,56 @@
       <mu2>0.8</mu2>
     </gazebo>
-    <gazebo reference="${prefix}lidar_link">
+    <gazebo reference="${prefix}ultrasonic_link">
       <material>Gazebo/Red</material>
+    </gazebo>
+    <!-- Ground-truth Odometry (P3D) -->
+    <gazebo>
+      <plugin name="gazebo_ros_ground_truth_odom" filename="libgazebo_ros_p3d.so">
+        <bodyName>${prefix}base_link</bodyName>
+        <topicName>/gazebo/odom_clean</topicName>
+        <frameName>world</frameName>
+        <xyzOffsets>0 0 0</xyzOffsets>
+        <rpyOffsets>0 0 0</rpyOffsets>
+        <updateRate>50.0</updateRate>
+        <gaussianNoise>0.0</gaussianNoise>
+      </plugin>
+    </gazebo>
+    <!-- Ultrasonic Range Sensor (HC-SR04 emulation) -->
+    <gazebo reference="${prefix}ultrasonic_link">
+      <sensor type="ray" name="ultrasonic_sensor">
+        <pose>0 0 0 0 0 0</pose>
+        <visualize>true</visualize>
+        <update_rate>20</update_rate>
+        <ray>
+          <scan>
+            <horizontal>
+              <samples>1</samples>
+              <resolution>1</resolution>
+              <min_angle>-0.13</min_angle>
+              <max_angle>0.13</max_angle>
+            </horizontal>
+          </scan>
+          <range>
+            <min>0.02</min>
+            <max>3.0</max>
+            <resolution>0.01</resolution>
+          </range>
+          <noise>
+            <type>gaussian</type>
+            <mean>0.0</mean>
+            <stddev>0.005</stddev>
+          </noise>
+        </ray>
+        <plugin name="ultrasonic_range_controller" filename="libgazebo_ros_range.so">
+          <topicName>/gazebo/ultrasonic_clean</topicName>
+          <frameName>${prefix}ultrasonic_link</frameName>
+          <radiationType>ultrasonic</radiationType>
+          <fov>0.26</fov>
+          <minDistance>0.02</minDistance>
+          <maxDistance>3.0</maxDistance>
+          <gaussianNoise>0.005</gaussianNoise>
+          <updateRate>20</updateRate>
+        </plugin>
+      </sensor>
     </gazebo>
   </xacro:if>

Commit message: fix: robot kinematics, planning stability, and occupancy grid reset
- cmd_vel_to_gazebo: rewrite to integrate twist into world-frame pose
  (bypasses ODE friction damping — actual velocity now matches commanded)
- navigation_manager: remove start_time reset on path_callback
  (goal timeout now works correctly)
- global_planner: add replan_distance check (0.5m)
  (reduces path thrashing, only replans when robot moves enough)
- URDF: reduce mass 15→2 kg, friction mu 0.8→0.02
  (lower inertia + less friction for Gazebo SetModelState)
- occupancy_grid: reset map on new goal via /mechdog/goal subscriber
  (prevents A* failure from accumulated occupied cells)
- simulation.launch: cmd_vel_to_gazebo rate 50→100 Hz
  (launch was overriding node default back to 50)

File: catkin_ws/src/mechdog_description/urdf/mechdog.urdf.xacro (robot description, xacro)
@@ -6,5 +6,5 @@
   <xacro:property name="robot_width" value="0.3"/>
   <xacro:property name="robot_height" value="0.2"/>
-  <xacro:property name="robot_mass" value="15.0"/>
+  <xacro:property name="robot_mass" value="2.0"/>
   <!-- Sensor Offsets — Ultrasonic at front-center, past the legs -->
   <xacro:property name="ultrasonic_offset_x" value="0.28"/>

File: catkin_ws/src/mechdog_description/urdf/mechdog_gazebo.xacro (robot description, xacro)
@@ -8,6 +8,6 @@
     <gazebo reference="${prefix}base_link">
       <material>Gazebo/Blue</material>
-      <mu1>0.8</mu1>
-      <mu2>0.8</mu2>
+      <mu1>0.02</mu1>
+      <mu2>0.02</mu2>
     </gazebo>
     <gazebo reference="${prefix}ultrasonic_link">
